File: Genesis rom edge connector only/Genesis rom edge connector only.kicad_pcb (KiCad board)
At the start: 2 copper layers, 104.1 x 29.4 mm, 6 parts, among them J1 Conn_01x32_Male, J2 Conn_01x32_Male, J3 Conn_01x32_Male, J4 Conn_01x32_Male

Commit message: basic flash functions are working
Finished implementing basic flash functions: read byte, write byte, erase  all, check mem type.
Fixed silk screen typo on pcb.
Other:
- board text added: "D13"
Changed lines of the file:
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@@
     (links 64)
     (no_connects 0)
-    (area 86.309999 69.357142 190.550001 103.92)
+    (area 86.309999 69.357142 190.550001 100.872)
     (thickness 1.6)
     (drawings 79)
@@
     (effects (font (size 1.5 1.5) (thickness 0.15)))
   )
-  (gr_text D14 (at 157.48 87.376 90) (layer F.SilkS)
+  (gr_text D13 (at 157.48 87.376 90) (layer F.SilkS)
     (effects (font (size 1.5 1.5) (thickness 0.15)))
   )
